Commit message: floribot_simulation migriert mit Fehler

File: ros1_ws/src/floribot_simulation/urdf/Floribot_reduced.urdf.xacro (robot description, xacro)
@@ -32,6 +32,4 @@
 <xacro:property name="wheel_joint_2_mid_joint" value="0.383" />
 <xacro:property name="joint_height" value="0.015" />
-<!-- add laserscanners -->
-<xacro:include filename="$(find sick_scan)/urdf/sick_scan.urdf.xacro" />
 <!-- macro wheel tranmission -->
 <xacro:macro name="wheel_transmission" params="position">

File: ros2_ws/src/floribot_simulation/urdf/Floribot_reduced.urdf.xacro (robot description, xacro)
@@ -1,4 +1,6 @@
 <?xml version="1.0" encoding="UTF-8"?>
-<robot xmlns:xacro="http://www.ros.org/wiki/xacro" name="Floribot">
+<robot xmlns:xacro="http://www.ros.org/wiki/xacro" xmlns:controller="http://playerstage.sourceforge.net/gazebo/xmlschema/#controller"
+  xmlns:interface="http://playerstage.sourceforge.net/gazebo/xmlschema/#interface"
+  xmlns:sensor="http://playerstage.sourceforge.net/gazebo/xmlschema/#sensor" name="Floribot">
 <!-- wagon parameter -->
 <xacro:property name="height_wagon" value="0.363" />
@@ -100,5 +102,5 @@
     <axis xyz="0 0 0"/>
     <geometry>
-      <mesh filename="package://floribot_simulation/meshes/Vorderwagen.stl" scale="0.001 0.001 0.001" />
+      <mesh filename="$(find floribot_simulation)/meshes/Vorderwagen.stl" scale="0.001 0.001 0.001" />
     </geometry>
     <material name="c">
@@ -282,5 +284,5 @@
     <axis xyz="0 0 0"/>
     <geometry>
-      <mesh filename="package://floribot_simulation/meshes/Hinterwagen.stl" scale="0.001 0.001 0.001" />
+      <mesh filename="$(find floribot_simulation)/meshes/Hinterwagen.stl" scale="0.001 0.001 0.001" />
     </geometry>
     <material name="b">
@@ -337,5 +339,5 @@
     <axis xyz="0 0 0"/>
     <geometry>
-      <mesh filename="package://floribot_simulation/meshes/Reifen.stl" scale="0.001 0.001 0.001" />
+      <mesh filename="$(find floribot_simulation)/meshes/Reifen.stl" scale="0.001 0.001 0.001" />
     </geometry>
     <material name="r">
@@ -370,5 +372,5 @@
     <axis xyz="0 0 0"/>
     <geometry>
-      <mesh filename="package://floribot_simulation/meshes/Reifen.stl" scale="0.001 0.001 0.001" />
+      <mesh filename="$(find floribot_simulation)/meshes/Reifen.stl" scale="0.001 0.001 0.001" />
     </geometry>
     <material name="r">
@@ -403,5 +405,5 @@
     <axis xyz="0 0 0"/>
     <geometry>
-      <mesh filename="package://floribot_simulation/meshes/Reifen.stl" scale="0.001 0.001 0.001" />
+      <mesh filename="$(find floribot_simulation)/meshes/Reifen.stl" scale="0.001 0.001 0.001" />
     </geometry>
     <material name="r">
@@ -436,5 +438,5 @@
     <axis xyz="0 0 0"/>
     <geometry>
-      <mesh filename="package://floribot_simulation/meshes/Reifen.stl" scale="0.001 0.001 0.001" />
+      <mesh filename="$(find floribot_simulation)/meshes/Reifen.stl" scale="0.001 0.001 0.001" />
     </geometry>
     <material name="r">
@@ -458,8 +460,32 @@
 <xacro:wheel_color linkName="rearLeft" />
 <xacro:wheel_color linkName="rearRight" />
-<!-- Gazebo plugin for ROS Control -->
+<ros2_control name="IgnitionSystem" type="system">
+  <hardware>
+    <plugin>ign_ros2_control/IgnitionSystem</plugin>
+  </hardware>
+  <joint name="joint_frontLeft">
+      <command_interface name="velocity" />
+      <state_interface name="velocity" />
+      <state_interface name="position" />
+  </joint>
+  <joint name="joint_frontRight">
+      <command_interface name="velocity" />
+      <state_interface name="velocity" />
+      <state_interface name="position" />
+  </joint>
+  <joint name="joint_rearLeft">
+      <command_interface name="velocity" />
+      <state_interface name="velocity" />
+      <state_interface name="position" />
+  </joint>
+  <joint name="joint_rearRight">
+      <command_interface name="velocity" />
+      <state_interface name="velocity" />
+      <state_interface name="position" />
+  </joint>
+</ros2_control>
 <gazebo>
-  <plugin name="gazebo_ros_control" filename="libgazebo_ros_control.so">
-    <!-- <robotNamespace>floribot</robotNamespace> -->
+  <plugin filename="ign_ros2_control-system" name="ign_ros2_control::IgnitionROS2ControlPlugin">
+    <parameters>$(find floribot_simulation)/config/joints.yaml</parameters>
   </plugin>
 </gazebo>
